File: pico_spi_adapter.kicad_sch (KiCad schematic)
At the start: 0 parts

Commit message: added components
Parts:
- added J1: Conn_01x02_Pin, symbol Connector:Conn_01x02_Pin
- added J2, J3: Conn_01x12_Socket, Connector_PinSocket_2.54mm:PinSocket_1x12_P2.54mm_Vertical, symbol Connector:Conn_01x12_Socket
- added J4: DE9_Receptacle, symbol Connector:DE9_Receptacle
- added U1: RaspberryPi_Pico, Module_RaspberryPi_Pico:RaspberryPi_Pico_Common, symbol ZhuLib:RaspberryPi_Pico
- added U2: MAX485CSA+T, 21-0041-3-M_90-0096-8L_MXM, symbol ZhuLib:MAX485CSA+T
Connections:
- new net +3.3V: J2.1 (Pin_1), J2.2 (Pin_2)
- new net +5V: J1.1 (Pin_1), U1.39 (VSYS), U2.8 (VCC)
- new net CS: J3.7 (Pin_7), U1.7 (GPIO5)
- new net GND: J1.2 (Pin_2), J3.1 (Pin_1), U1.13 (GND), U1.18 (GND), U1.23 (GND), U1.28 (GND), U1.3 (GND), U1.33 (AGND), U1.38 (GND), U1.8 (GND), U2.5 (GND)
- new net INT1: J3.2 (Pin_2)
- new net INT2: J3.3 (Pin_3)
- new net MISO: J3.9 (Pin_9), U1.6 (GPIO4)
- new net MOSI: J3.10 (Pin_10), U1.5 (GPIO3)
- new net SCK: J3.8 (Pin_8), U1.4 (GPIO2)

Commit message: added a few things
Parts:
- added J5: Screw_Terminal_01x02, symbol Connector:Screw_Terminal_01x02
- added R1: 120, symbol Device:R
Connections:
- net +3.3V: now also U1.36 (3V3)
- net +5V: now also J5.1 (Pin_1)
- net GND: now also J4.5, J5.2 (Pin_2)
- net INT1: now also U1.20 (GPIO15)
- net INT2: now also U1.21 (GPIO16)
- net UART_TX: now reaches U1.11 (GPIO8)
- net UART_TX: now also U2.4 (DI)
- net UART_RX: now reaches U1.12 (GPIO9)
- net UART_RX: now also U2.1 (RO)
- net RST: now reaches U1.29 (GPIO22)
- net RST: now also U2.2 (*RE), U2.3 (DE)
- net RS485_B: now reaches U2.6 (A)
- net RS485_B: now also J4.2, R1.2
- net RS485_A: now reaches U2.7 (B)
- net RS485_A: now also J4.3, R1.1
- no-connect marks 0 -> 18
Other:
- note added: "12V - 5V DCDC"
- note added: "ASM330LHH Connector"
- note added: "NRU-230V-AWP RS485_DATA-, Pin 3 RS485_DATA+, Pin 2 RS485_GND, Pin 5"
- note added: "RS485 Connector"
- note added: "RS485 Levelshifter"
- note added: "Raspberry Pi Pico"
- moved on the sheet: J1, J2, J3, J4, U1, U2

Commit message: added buck ic, updated layout
Parts:
- added U3: TPS5405DR, D0008A-IPC_A, symbol ZhuLib:TPS5405DR
Changed lines of the file:
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@@
+    )
+  )
+  (symbol (lib_id "ZhuLib:TPS5405DR") (at 220.345 114.935 0) (unit 1)
+    (in_bom yes) (on_board yes) (dnp no) (fields_autoplaced)
+    (property "Reference" "U3" (at 240.665 105.8006 0)
+      (effects (font (size 1.524 1.524)))
+    )
+    (property "Value" "TPS5405DR" (at 240.665 108.1818 0)
+      (effects (font (size 1.524 1.524)))
+    )
+    (property "Footprint" "D0008A-IPC_A" (at 217.805 135.255 0)
+      (effects (font (size 1.27 1.27) italic) hide)
+    )
+    (property "Datasheet" "https://www.ti.com/lit/gpn/tps5405" (at 212.725 137.795 0)
+      (effects (font (size 1.27 1.27) italic) hide)
+    )
+    (pin "1")
+    (pin "2")
+    (pin "3")
+    (pin "4")
+    (pin "5")
+    (pin "6")
+    (pin "7")
+    (pin "8")
+    (instances
+      (project "pico_spi_adapter"
+        (path "/4ab7442f-0fdf-4059-bb07-5c2df8059f04"
+          (reference "U3") (unit 1)
+        )
+      )
     )
   )

Commit message: added parts
Parts:
- added C1: C, Capacitor_SMD:C_1206_3216Metric, symbol Device:C
- added C2, C4, C5: C, symbol Device:C
- added C3: 0.1u, Resistor_SMD:R_1206_3216Metric, symbol Device:C
- added D1: 1N5712, Diode_THT:D_DO-35_SOD27_P7.62mm_Horizontal, symbol Diode:1N5712
- added L1: L, ZhuLib:IND_-B953AS-100M=P3_MUR, symbol Device:L
- added R2: R, symbol Device:R
- added R3: 85.5k, symbol Device:R
Connections:
- net +5V: now also C4.2, L1.2; no longer J5.1 (Pin_1)
- net GND: now also U3.7 (GND), C1.2, C2.2, C4.1, C5.2, D1.2 (A), R3.2
- net at U3.1 (BOOT): now also C3.1
- net +12V: now reaches U3.2 (VIN)
- net +12V: now also C5.1
- net at U3.3 (ROSC): now also R3.1
- net at U3.4 (SS): now also C1.1
- net at U3.5 (VSENSE): now also U3.8 (LX), C3.2, D1.1 (K), L1.1
- net at U3.6 (COMP): now also R2.1
- new net: C2.1, R2.2
- new net Vin: J5.1 (Pin_1)
Other:
- moved on the sheet: J1, J5, U3

Commit message: added calc & part selections.
Parts:
- removed J1: Conn_01x02_Pin, symbol Connector:Conn_01x02_Pin
- removed J5: Screw_Terminal_01x02, symbol Connector:Screw_Terminal_01x02
- added D3: ~, symbol Diode:1N5712
- D1: value 1N5712 -> ~; footprint Diode_THT:D_DO-35_SOD27_P7.62mm_Horizontal -> (none); JLCPCB Part# (none) -> C47460
- L1: value L -> 33uH; footprint ZhuLib:IND_-B953AS-100M=P3_MUR -> (none); JLCPCB Part# C2047362 -> C2847546
- R3: footprint (none) -> Resistor_SMD:R_0805_2012Metric; JLCPCB Part# (none) -> C17842
Connections:
- net +12V: now also J4.1, D3.2 (A); no longer C5.1, U3.2 (VIN)
- net Vsense: now reaches C3.2, D1.1 (K), L1.1, U3.5 (VSENSE), U3.8 (LX)
- new net: C5.1, D3.1 (K), U3.2 (VIN)
- no-connect marks 18 -> 23
Other:
- moved on the sheet: C1, C2, C3, C4, C5, D1, L1, R1, R2, R3, U2, U3

Commit message: updated layouts
Parts:
- removed D3: ~, symbol Diode:1N5712
- added D1: ~, symbol Diode:1N5712
- added D3: LED, LED_SMD:LED_0201_0603Metric, symbol Device:LED
- added J3: Conn_01x06_Pin, symbol Connector:Conn_01x06_Pin
- added J4: Screw_Terminal_01x02, TerminalBlock_Phoenix:TerminalBlock_Phoenix_MPT-0,5-2-2.54_1x02_P2.54mm_Horizontal, symbol Connector:Screw_Terminal_01x02
- added R4: 150, Resistor_SMD:R_0805_2012Metric, symbol Device:R
- C1: renamed from C5; value C -> 10uF; footprint (none) -> Capacitor_SMD:C_0805_2012Metric; JLCPCB Part# (none) -> C15850
- C2: renamed from C1; value C -> 12nF
- C3: renamed from C2; value C -> 4.7nF; footprint (none) -> Capacitor_SMD:C_0805_2012Metric; JLCPCB Part# (none) -> C50131
- C4: renamed from C3; value 0.1u -> 0.1uF; footprint Resistor_SMD:R_1206_3216Metric -> Capacitor_SMD:C_0805_2012Metric; JLCPCB Part# C24497 -> C1711
- C5: renamed from C4; value C -> 22uF; footprint (none) -> Capacitor_SMD:C_0805_2012Metric; JLCPCB Part# (none) -> C5674
- J5: renamed from J4; footprint (none) -> Connector_Dsub:DSUB-9_Female_Horizontal_P2.77x2.84mm_EdgePinOffset14.56mm_Housed_MountingHolesOffset15.98mm
- L1: footprint (none) -> Inductor_SMD:L_Wuerth_HCM-7050
- R2: value R -> 10k; footprint (none) -> Resistor_SMD:R_0805_2012Metric; JLCPCB Part# (none) -> C100047
- R3: value 85.5k -> 84.5k
- U3: footprint D0008A-IPC_A -> ZhuLib:21-0041-3-M_90-0096-8L_MXM
- renumbered D1 to D2, J2 to J1, J3 to J2
Connections:
- net +12V: now also D1.2 (A), J3.1 (Pin_1)
- net +5V: now also U3.5 (VSENSE), J3.2 (Pin_2), J4.1 (Pin_1), R4.1
- net GND: now also D3.1 (K), J3.4 (Pin_4), J3.5 (Pin_5), J3.6 (Pin_6), J4.2 (Pin_2)
- net RS485_A: now also R1.2, U2.6 (A); no longer R1.1, U2.7 (B)
- net RS485_B: now also R1.1, U2.7 (B); no longer R1.2, U2.6 (A)
- net at C1.1, U3.2 (VIN): now also D1.1 (K)
- net Vsense: no longer names the net of C4.2, D2.1 (K), L1.1, U3.8 (LX)
- net Vsense: no longer U3.5 (VSENSE)
- new net: D3.2 (A), R4.2
- no-connect marks 23 -> 42
Other:
- title: (none) -> Pico asm330lhh adapter board
- moved on the sheet: C5, D2, L1

Commit message: layout size
Parts:
- added H1, H2, H3, H4: MountingHole, MountingHole:MountingHole_3.2mm_M3_DIN965_Pad, symbol Mechanical:MountingHole_Pad
- J3: footprint (none) -> Connector_PinHeader_2.54mm:PinHeader_1x06_P2.54mm_Vertical
Connections:
- net GND: now also H1.1, H2.1, H3.1, H4.1
Changed lines of the file:
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@@
+    )
+  )
+  (symbol (lib_id "power:GND") (at 148.59 49.53 0) (unit 1)
+    (in_bom yes) (on_board yes) (dnp no) (fields_autoplaced)
+    (property "Reference" "#PWR027" (at 148.59 55.88 0)
+      (effects (font (size 1.27 1.27)) hide)
+    )
+    (property "Value" "GND" (at 148.59 54.61 0)
+      (effects (font (size 1.27 1.27)))
+    )
+    (property "Footprint" "" (at 148.59 49.53 0)
+      (effects (font (size 1.27 1.27)) hide)
+    )
+    (property "Datasheet" "" (at 148.59 49.53 0)
+      (effects (font (size 1.27 1.27)) hide)
+    )
+    (pin "1")
+    (instances
+      (project "pico_spi_adapter"
+        (path "/4ab7442f-0fdf-4059-bb07-5c2df8059f04"
+          (reference "#PWR027") (unit 1)
+        )
+      )
     )
   )
@@
     )
   )
+  (symbol (lib_id "power:GND") (at 161.29 49.53 0) (unit 1)
+    (in_bom yes) (on_board yes) (dnp no) (fields_autoplaced)
+    (property "Reference" "#PWR029" (at 161.29 55.88 0)
+      (effects (font (size 1.27 1.27)) hide)
+    )
+    (property "Value" "GND" (at 161.29 54.61 0)
+      (effects (font (size 1.27 1.27)))
+    )
+    (property "Footprint" "" (at 161.29 49.53 0)
+      (effects (font (size 1.27 1.27)) hide)
+    )
+    (property "Datasheet" "" (at 161.29 49.53 0)
+      (effects (font (size 1.27 1.27)) hide)
+    )
+    (pin "1")
+    (instances
+      (project "pico_spi_adapter"
+        (path "/4ab7442f-0fdf-4059-bb07-5c2df8059f04"
+          (reference "#PWR029") (unit 1)
+        )
+      )
+    )
+  )
   (symbol (lib_id "Device:C") (at 234.95 110.49 90) (unit 1)
     (in_bom yes) (on_board yes) (dnp no) (fields_autoplaced)
@@
       (effects (font (size 1.27 1.27)) hide)
     )
-    (property "Footprint" "" (at 114.3 111.76 0)
+    (property "Footprint" "Connector_PinHeader_2.54mm:PinHeader_1x06_P2.54mm_Vertical" (at 114.3 111.76 0)
       (effects (font (size 1.27 1.27)) hide)
     )
@@
     )
   )
+  (symbol (lib_id "Mechanical:MountingHole_Pad") (at 148.59 46.99 0) (unit 1)
+    (in_bom yes) (on_board yes) (dnp no) (fields_autoplaced)
+    (property "Reference" "H1" (at 151.13 45.72 0)
+      (effects (font (size 1.27 1.27)) (justify left))
+    )
+    (property "Value" "MountingHole" (at 151.13 48.26 0)
+      (effects (font (size 1.27 1.27)) (justify left))
+    )
+    (property "Footprint" "MountingHole:MountingHole_3.2mm_M3_DIN965_Pad" (at 148.59 46.99 0)
+      (effects (font (size 1.27 1.27)) hide)
+    )
+    (property "Datasheet" "~" (at 148.59 46.99 0)
+      (effects (font (size 1.27 1.27)) hide)
+    )
+    (pin "1")
+    (instances
+      (project "pico_spi_adapter"
+        (path "/4ab7442f-0fdf-4059-bb07-5c2df8059f04"
+          (reference "H1") (unit 1)
+        )
+      )
+    )
+  )
   (symbol (lib_id "Device:R") (at 111.76 39.37 0) (unit 1)
     (in_bom yes) (on_board yes) (dnp no)
@@
         (path "/4ab7442f-0fdf-4059-bb07-5c2df8059f04"
           (reference "#PWR022") (unit 1)
+        )
+      )
+    )
+  )
+  (symbol (lib_id "Mechanical:MountingHole_Pad") (at 154.94 46.99 0) (unit 1)
+    (in_bom yes) (on_board yes) (dnp no) (fields_autoplaced)
+    (property "Reference" "H2" (at 157.48 45.72 0)
+      (effects (font (size 1.27 1.27)) (justify left))
+    )
+    (property "Value" "MountingHole" (at 157.48 48.26 0)
+      (effects (font (size 1.27 1.27)) (justify left))
+    )
+    (property "Footprint" "MountingHole:MountingHole_3.2mm_M3_DIN965_Pad" (at 154.94 46.99 0)
+      (effects (font (size 1.27 1.27)) hide)
+    )
+    (property "Datasheet" "~" (at 154.94 46.99 0)
+      (effects (font (size 1.27 1.27)) hide)
+    )
+    (pin "1")
+    (instances
+      (project "pico_spi_adapter"
+        (path "/4ab7442f-0fdf-4059-bb07-5c2df8059f04"
+          (reference "H2") (unit 1)
         )
       )
@@
     )
   )
+  (symbol (lib_id "Mechanical:MountingHole_Pad") (at 161.29 46.99 0) (unit 1)
+    (in_bom yes) (on_board yes) (dnp no) (fields_autoplaced)
+    (property "Reference" "H3" (at 163.83 45.72 0)
+      (effects (font (size 1.27 1.27)) (justify left))
+    )
+    (property "Value" "MountingHole" (at 163.83 48.26 0)
+      (effects (font (size 1.27 1.27)) (justify left))
+    )
+    (property "Footprint" "MountingHole:MountingHole_3.2mm_M3_DIN965_Pad" (at 161.29 46.99 0)
+      (effects (font (size 1.27 1.27)) hide)
+    )
+    (property "Datasheet" "~" (at 161.29 46.99 0)
+      (effects (font (size 1.27 1.27)) hide)
+    )
+    (pin "1")
+    (instances
+      (project "pico_spi_adapter"
+        (path "/4ab7442f-0fdf-4059-bb07-5c2df8059f04"
+          (reference "H3") (unit 1)
+        )
+      )
+    )
+  )
   (symbol (lib_id "power:GND") (at 55.88 175.26 0) (unit 1)
     (in_bom yes) (on_board yes) (dnp no) (fields_autoplaced)
@@
     )
   )
+  (symbol (lib_id "Mechanical:MountingHole_Pad") (at 167.64 46.99 0) (unit 1)
+    (in_bom yes) (on_board yes) (dnp no) (fields_autoplaced)
+    (property "Reference" "H4" (at 170.18 45.72 0)
+      (effects (font (size 1.27 1.27)) (justify left))
+    )
+    (property "Value" "MountingHole" (at 170.18 48.26 0)
+      (effects (font (size 1.27 1.27)) (justify left))
+    )
+    (property "Footprint" "MountingHole:MountingHole_3.2mm_M3_DIN965_Pad" (at 167.64 46.99 0)
+      (effects (font (size 1.27 1.27)) hide)
+    )
+    (property "Datasheet" "~" (at 167.64 46.99 0)
+      (effects (font (size 1.27 1.27)) hide)
+    )
+    (pin "1")
+    (instances
+      (project "pico_spi_adapter"
+        (path "/4ab7442f-0fdf-4059-bb07-5c2df8059f04"
+          (reference "H4") (unit 1)
+        )
+      )
+    )
+  )
   (symbol (lib_id "power:+5V") (at 256.54 128.27 0) (unit 1)
     (in_bom yes) (on_board yes) (dnp no) (fields_autoplaced)
@@
         )
       )
+    )
+  )
+  (symbol (lib_id "power:GND") (at 154.94 49.53 0) (unit 1)
+    (in_bom yes) (on_board yes) (dnp no) (fields_autoplaced)
+    (property "Reference" "#PWR028" (at 154.94 55.88 0)
+      (effects (font (size 1.27 1.27)) hide)
+    )
+    (property "Value" "GND" (at 154.94 54.61 0)
+      (effects (font (size 1.27 1.27)))
+    )
+    (property "Footprint" "" (at 154.94 49.53 0)
+      (effects (font (size 1.27 1.27)) hide)
+    )
+    (property "Datasheet" "" (at 154.94 49.53 0)
+      (effects (font (size 1.27 1.27)) hide)
+    )
+    (pin "1")
+    (instances
+      (project "pico_spi_adapter"
+        (path "/4ab7442f-0fdf-4059-bb07-5c2df8059f04"
+          (reference "#PWR028") (unit 1)
+        )
+      )
+    )
+  )
+  (symbol (lib_id "power:GND") (at 167.64 49.53 0) (unit 1)
+    (in_bom yes) (on_board yes) (dnp no) (fields_autoplaced)
+    (property "Reference" "#PWR030" (at 167.64 55.88 0)
+      (effects (font (size 1.27 1.27)) hide)
+    )
+    (property "Value" "GND" (at 167.64 54.61 0)
+      (effects (font (size 1.27 1.27)))
+    )
+    (property "Footprint" "" (at 167.64 49.53 0)
+      (effects (font (size 1.27 1.27)) hide)
+    )
+    (property "Datasheet" "" (at 167.64 49.53 0)
+      (effects (font (size 1.27 1.27)) hide)
+    )
+    (pin "1")
+    (instances
+      (project "pico_spi_adapter"
+        (path "/4ab7442f-0fdf-4059-bb07-5c2df8059f04"
+          (reference "#PWR030") (unit 1)
+        )
+      )

Commit message: added a step file
Parts:
- D1, D2: footprint (none) -> Diode_SMD:D_SMA
- R1: footprint (none) -> Resistor_SMD:R_0805_2012Metric; JLCPCB PART# (none) -> C17437
Changed lines of the file:
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@@
       (effects (font (size 1.27 1.27)) (justify left))
     )
-    (property "Footprint" "" (at 240.665 115.57 0)
+    (property "Footprint" "Diode_SMD:D_SMA" (at 240.665 115.57 0)
       (effects (font (size 1.27 1.27)) hide)
     )
@@
   )
   (symbol (lib_id "Mechanical:MountingHole_Pad") (at 148.59 46.99 0) (unit 1)
-    (in_bom yes) (on_board yes) (dnp no) (fields_autoplaced)
-    (property "Reference" "H1" (at 151.13 45.72 0)
+    (in_bom yes) (on_board yes) (dnp no)
+    (property "Reference" "H1" (at 147.32 41.91 0)
       (effects (font (size 1.27 1.27)) (justify left))
     )
     (property "Value" "MountingHole" (at 151.13 48.26 0)
-      (effects (font (size 1.27 1.27)) (justify left))
+      (effects (font (size 1.27 1.27)) (justify left) hide)
     )
     (property "Footprint" "MountingHole:MountingHole_3.2mm_M3_DIN965_Pad" (at 148.59 46.99 0)
@@
       (effects (font (size 1.27 1.27)) (justify left))
     )
-    (property "Footprint" "" (at 109.982 39.37 90)
+    (property "Footprint" "Resistor_SMD:R_0805_2012Metric" (at 109.982 39.37 90)
       (effects (font (size 1.27 1.27)) hide)
     )
@@
       (effects (font (size 1.27 1.27)) hide)
     )
+    (property "JLCPCB PART#" "C17437" (at 111.76 39.37 0)
+      (effects (font (size 1.27 1.27)) hide)
+    )
     (pin "1")
     (pin "2")
@@
   )
   (symbol (lib_id "Mechanical:MountingHole_Pad") (at 154.94 46.99 0) (unit 1)
-    (in_bom yes) (on_board yes) (dnp no) (fields_autoplaced)
-    (property "Reference" "H2" (at 157.48 45.72 0)
+    (in_bom yes) (on_board yes) (dnp no)
+    (property "Reference" "H2" (at 153.67 41.91 0)
       (effects (font (size 1.27 1.27)) (justify left))
     )
     (property "Value" "MountingHole" (at 157.48 48.26 0)
-      (effects (font (size 1.27 1.27)) (justify left))
+      (effects (font (size 1.27 1.27)) (justify left) hide)
     )
     (property "Footprint" "MountingHole:MountingHole_3.2mm_M3_DIN965_Pad" (at 154.94 46.99 0)
@@
       (effects (font (size 1.27 1.27)) (justify left))
     )
-    (property "Footprint" "" (at 169.545 104.14 0)
+    (property "Footprint" "Diode_SMD:D_SMA" (at 169.545 104.14 0)
       (effects (font (size 1.27 1.27)) hide)
     )
@@
   )
   (symbol (lib_id "Mechanical:MountingHole_Pad") (at 161.29 46.99 0) (unit 1)
-    (in_bom yes) (on_board yes) (dnp no) (fields_autoplaced)
-    (property "Reference" "H3" (at 163.83 45.72 0)
+    (in_bom yes) (on_board yes) (dnp no)
+    (property "Reference" "H3" (at 160.02 41.91 0)
       (effects (font (size 1.27 1.27)) (justify left))
     )
     (property "Value" "MountingHole" (at 163.83 48.26 0)
-      (effects (font (size 1.27 1.27)) (justify left))
+      (effects (font (size 1.27 1.27)) (justify left) hide)
     )
     (property "Footprint" "MountingHole:MountingHole_3.2mm_M3_DIN965_Pad" (at 161.29 46.99 0)
@@
   )
   (symbol (lib_id "Mechanical:MountingHole_Pad") (at 167.64 46.99 0) (unit 1)
-    (in_bom yes) (on_board yes) (dnp no) (fields_autoplaced)
-    (property "Reference" "H4" (at 170.18 45.72 0)
-      (effects (font (size 1.27 1.27)) (justify left))
-    )
+    (in_bom yes) (on_board yes) (dnp no)
+    (property "Reference" "H4" (at 166.37 41.91 0)
+      (effects (font (size 1.27 1.27)) (justify left))
+    )
